File: uaefi-adapter.kicad_sch (KiCad schematic)
At the start: 14 parts, among them J1 43045-0612, J2 43045-0412, J2 43045-0612, J3 43045-0612, J4 43045-0212, M1 Module:uaefi/0.2, P3 Pad, P30 Pad, P32 Pad, P4 Pad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

Commit message: #1
Connections:
- net ETB_N: no longer M1.A1 (OUT_DC1-)
- net ETB_P: no longer M1.A5 (OUT_DC1+)
- net AC RELAY: no longer names the net of M1.B18 (OUT_LS2)
- net AUX1: no longer names the net of M1.D1 (IN_AUX1)
- net AUX3: no longer names the net of M1.C15 (IN_AUX3)
- net BTN3: no longer names the net of M1.C9 (IN_BUTTON3)
- net BUTTON1: no longer names the net of M1.D2 (IN_BUTTON1)
- net DC2+: no longer names the net of M1.A6 (OUT_DC2+)
- net Engine_Light: no longer names the net of M1.B8 (OUT_LS_HOT2)
- net HALL3: no longer names the net of M1.C7 (IN_HALL3)
- net IN_CAM1_POS: no longer names the net of M1.C6 (IN_HALL2)
- net IN_CRANK_VR: no longer names the net of M1.C5 (IN_HALL1)
- net IN_HS_BRAKE: no longer names the net of M1.D10 (IN_BUTTON2)
- net IN_KNOCK: no longer names the net of M1.D14 (IN_KNOCK_RAW)
- net IN_MAP: no longer names the net of M1.D9 (IN_MAP)
- net Intake_Bypass_VSV1: no longer names the net of M1.B17 (OUT_LS3)
- net MAF: no longer names the net of M1.C3 (IN_AUX2)
- net OUT_IGN5: no longer names the net of M1.B13 (OUT_IGN5)
- net OUT_IGN6: no longer names the net of M1.B10 (OUT_IGN6)
- net OUT_INJ5: no longer names the net of M1.B2 (OUT_INJ5)
- net OUT_INJ6: no longer names the net of M1.B1 (OUT_INJ6)
- net TACHO: no longer names the net of M1.B9 (OUT_LS_HOT1)
- net VR1+: no longer names the net of M1.C18 (VR_DISCRETE+)
- net VR1-: no longer names the net of M1.C19 (VR_DISCRETE-)
- net VR2+: no longer names the net of M1.C16 (VR_MAX9924+)
- net VR2-: no longer names the net of M1.C17 (VR_MAX9924-)
- net Wastegate_Control: no longer names the net of M1.B7 (OUT_LS1)

Commit message: #2
Connections:
- net ETB_N: now also M1.A1 (OUT_DC1-)
- net ETB_P: now also M1.A5 (OUT_DC1+)
Changed lines of the file:
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@@
+    (stroke (width 0) (type default))
+  )
+  (bus_entry (at 182.245 100.33) (size -2.54 2.54)
     (stroke (width 0) (type default))
   )
@@
     (stroke (width 0) (type default))
   )
-  (bus_entry (at 179.705 135.89) (size -2.54 2.54)
+  (bus_entry (at 182.245 90.17) (size -2.54 2.54)
     (stroke (width 0) (type default))
   )
@@
     (stroke (width 0) (type default))
   )
-  (bus (pts (xy 172.085 237.49) (xy 172.085 247.65))
+  (bus (pts (xy 172.085 229.87) (xy 172.085 247.65))
     (stroke (width 0) (type default) (color 255 0 255 1))
   )
@@
     (stroke (width 0) (type default))
   )
-  (bus (pts (xy 172.085 250.19) (xy 172.085 252.73))
+  (wire (pts (xy 182.245 90.17) (xy 213.995 90.17))
+    (stroke (width 0) (type default))
+  )
+  (bus (pts (xy 172.085 247.65) (xy 172.085 252.73))
     (stroke (width 0) (type default) (color 255 0 255 1))
   )
@@
     (stroke (width 0) (type default))
   )
-  (bus (pts (xy 172.085 247.65) (xy 172.085 250.19))
-    (stroke (width 0) (type default) (color 255 0 255 1))
-  )
   (wire (pts (xy 174.625 227.33) (xy 213.995 227.33))
     (stroke (width 0) (type default))
@@
     (stroke (width 0) (type default))
   )
-  (bus (pts (xy 172.085 229.87) (xy 172.085 237.49))
-    (stroke (width 0) (type default) (color 255 0 255 1))
-  )
   (wire (pts (xy 155.575 70.485) (xy 161.925 70.485))
     (stroke (width 0) (type default))
@@
     (stroke (width 0) (type dash))
   )
+  (wire (pts (xy 182.245 100.33) (xy 213.995 100.33))
+    (stroke (width 0) (type default))
+  )
   (wire (pts (xy 202.565 290.83) (xy 202.565 285.75))
     (stroke (width 0) (type default))
@@
     (stroke (width 0) (type default))
   )
-  (wire (pts (xy 179.705 135.89) (xy 213.995 135.89))
-    (stroke (width 0) (type default))
-  )
   (bus (pts (xy 90.17 24.13) (xy 74.93 24.13))
     (stroke (width 0.3048) (type solid) (color 255 0 0 1))
@@
     (stroke (width 0) (type default) (color 255 0 255 1))
   )
-  (bus (pts (xy 164.465 73.025) (xy 177.165 73.025))
+  (bus (pts (xy 164.465 73.025) (xy 179.705 73.025))
+    (stroke (width 0) (type default) (color 0 194 194 1))
+  )
+  (bus (pts (xy 179.705 92.71) (xy 179.705 102.87))
     (stroke (width 0) (type default) (color 0 194 194 1))
   )
@@
   (bus (pts (xy 172.085 55.245) (xy 172.085 70.485))
     (stroke (width 0) (type default) (color 255 0 255 1))
+  )
+  (bus (pts (xy 179.705 73.025) (xy 179.705 92.71))
+    (stroke (width 0) (type default) (color 0 194 194 1))
   )
   (wire (pts (xy 172.085 285.75) (xy 172.085 295.91))
@@
     (effects (font (size 1.27 1.27)) (justify left bottom))
   )
+  (label "ETB_N" (at 188.595 90.17 0) (fields_autoplaced)
+    (effects (font (size 1.27 1.27)) (justify left bottom))
+  )
   (label "EGT+" (at 152.4 187.325 0) (fields_autoplaced)
     (effects (font (size 1.27 1.27)) (justify left bottom))
@@
     (effects (font (size 1.27 1.27)) (justify left bottom))
   )
+  (label "ETB_P" (at 194.31 100.33 180) (fields_autoplaced)
+    (effects (font (size 1.27 1.27)) (justify right bottom))
+  )
   (label "WBO_HTR-" (at 191.135 262.89 0) (fields_autoplaced)
